File: Hardware/ReflowController/TemperatureReader.kicad_sch (KiCad schematic)
At the start: 0 parts

Commit message: defined rough structure with kerem
Parts:
- added U4: MAX31865xAP, Package_SO:SSOP-20_5.3x7.2mm_P0.65mm, symbol Sensor_Temperature:MAX31865xAP
Connections:
- new net: U4.13 (GND), U4.19 (GND)
Changed lines of the file:
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@@
-(kicad_sch (version 20211123) (generator eeschema)
+(kicad_sch (version 20230121) (generator eeschema)
   (paper "A4")
-  (hierarchical_label "MOSI" (shape input) (at 104.14 92.71 0)
+  (hierarchical_label "CS" (shape input) (at 104.14 100.33 0) (fields_autoplaced)
     (effects (font (size 1.27 1.27)) (justify left))
   )
-  (hierarchical_label "SCLK" (shape input) (at 104.14 97.79 0)
+  (hierarchical_label "MOSI" (shape input) (at 104.14 92.71 0) (fields_autoplaced)
     (effects (font (size 1.27 1.27)) (justify left))
   )
-  (hierarchical_label "MISO" (shape output) (at 104.14 95.25 0)
+  (hierarchical_label "SCLK" (shape input) (at 104.14 97.79 0) (fields_autoplaced)
     (effects (font (size 1.27 1.27)) (justify left))
   )
-  (hierarchical_label "DGND" (shape passive) (at 116.84 106.68 0)
+  (hierarchical_label "MISO" (shape output) (at 104.14 95.25 0) (fields_autoplaced)
     (effects (font (size 1.27 1.27)) (justify left))
   )
-  (hierarchical_label "+5VD" (shape input) (at 116.84 102.87 0)
+  (hierarchical_label "DGND" (shape passive) (at 116.84 106.68 0) (fields_autoplaced)
     (effects (font (size 1.27 1.27)) (justify left))
   )
+  (hierarchical_label "+5VD" (shape input) (at 116.84 102.87 0) (fields_autoplaced)
+    (effects (font (size 1.27 1.27)) (justify left))
+  )
+  (symbol (lib_id "Sensor_Temperature:MAX31865xAP") (at 160.02 87.63 0) (unit 1)
+    (in_bom yes) (on_board yes) (dnp no) (fields_autoplaced)
+    (property "Reference" "U4" (at 164.5159 66.04 0)
+      (effects (font (size 1.27 1.27)) (justify left))
+    )
+    (property "Value" "MAX31865xAP" (at 164.5159 68.58 0)
+      (effects (font (size 1.27 1.27)) (justify left))
+    )
+    (property "Footprint" "Package_SO:SSOP-20_5.3x7.2mm_P0.65mm" (at 163.83 104.14 0)
+      (effects (font (size 1.27 1.27)) (justify left) hide)
+    )
+    (property "Datasheet" "https://datasheets.maximintegrated.com/en/ds/MAX31865.pdf" (at 160.02 80.01 0)
+      (effects (font (size 1.27 1.27)) hide)
+    )
+    (pin "1")
+    (pin "10")
+    (pin "11")
+    (pin "12")
+    (pin "13")
+    (pin "14")
+    (pin "15")
+    (pin "16")
+    (pin "17")
+    (pin "18")
+    (pin "19")
+    (pin "2")
+    (pin "20")
+    (pin "3")
+    (pin "4")
+    (pin "5")
+    (pin "6")
+    (pin "7")
+    (pin "8")
+    (pin "9")
+    (instances
+      (project "ReflowController"
+        (path "/2394cc2a-b9b0-4c0b-be11-1fc6085b0d5c/cedd135a-27b6-4ce6-9f5e-bdcd93291ccf"
+          (reference "U4") (unit 1)
+        )
+      )
+    )
+  )
 )

Commit message: started with schematic
Parts:
- added C1, C2: 100n, Capacitor_SMD:C_1206_3216Metric, symbol Device:C
- added NT2: NetTie_2, symbol Device:NetTie_2
- added R1: R, symbol Device:R
Connections:
- net DGND: now also U4.18 (DGND), C1.2, NT2.1
- net MISO: now also U4.17 (SDO)
- net MOSI: now also U4.14 (SDI)
- net SCLK: now also U4.15 (SCLK)
- net at U4.11 (RTDIN-): now also U4.12 (FORCE-)
- net AGND: now reaches U4.13 (GND), U4.19 (GND)
- net AGND: now also C2.2, NT2.2
- net ~{CS}: now reaches U4.16 (~{CS})
- net +3.3VD: now reaches U4.2 (DVDD)
- net +3.3VD: now also U4.3 (VDD), C1.1, C2.1
- net at U4.4 (BIAS): now also U4.5 (REFIN+), R1.1
- net at U4.6 (REFIN-): now also U4.7 (ISENSOR), R1.2
- net at U4.8 (FORCE+): now also U4.9 (FORCE2)
Other:
- note added: "TODO: - add protection diodes to all 4x wires - make a circuit with dipswitches to infrom system if 4x wire or 3x wire sense is used - figure out circuit to switch between PT100 and PT1000"
- note added: "analog GND plane connect"
- moved on the sheet: U4

Commit message: work on temp ic circuit
Parts:
- added C3: 10n, Capacitor_SMD:C_1206_3216Metric, symbol Device:C
- added NT3: NetTie_2, symbol Device:NetTie_2
- added TP1: T_RDY, symbol Connector:TestPoint
- R1: value R -> 402
Connections:
- net +3.3VD: now also NT3.2; no longer C2.1, U4.3 (VDD)
- net ~{DATA_READY}: now reaches U4.1 (~{DRDY})
- net ~{DATA_READY}: now also TP1.1
- net PT100_+IN: now reaches U4.10 (RTDIN+)
- net PT100_+IN: now also C3.2
- net PT100_-IN: now reaches U4.11 (RTDIN-), U4.12 (FORCE-)
- net PT100_-IN: now also C3.1
- net PT100_+OUT: now reaches U4.8 (FORCE+), U4.9 (FORCE2)
- new net: C2.1, NT3.1, U4.3 (VDD)
Changed lines of the file:
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@@
   (junction (at 154.94 99.06) (diameter 0) (color 0 0 0 0)
   )
+  (junction (at 190.5 82.55) (diameter 0) (color 0 0 0 0)
+  )
   (junction (at 170.18 77.47) (diameter 0) (color 0 0 0 0)
   )
@@
   (junction (at 170.18 90.17) (diameter 0) (color 0 0 0 0)
   )
+  (junction (at 190.5 93.98) (diameter 0) (color 0 0 0 0)
+  )
   (junction (at 170.18 62.23) (diameter 0) (color 0 0 0 0)
   )
+  (junction (at 114.3 62.23) (diameter 0) (color 0 0 0 0)
+  )
   (junction (at 149.86 50.8) (diameter 0) (color 0 0 0 0)
   )
@@
     (stroke (width 0) (type default))
   )
-  (wire (pts (xy 129.54 64.77) (xy 137.16 64.77))
+  (wire (pts (xy 101.6 64.77) (xy 137.16 64.77))
     (stroke (width 0) (type default))
   )
@@
     (stroke (width 0) (type default))
   )
+  (wire (pts (xy 190.5 82.55) (xy 190.5 83.82))
+    (stroke (width 0) (type default))
+  )
   (wire (pts (xy 149.86 95.25) (xy 149.86 109.22))
     (stroke (width 0) (type default))
@@
     (stroke (width 0) (type default))
   )
+  (wire (pts (xy 170.18 93.98) (xy 190.5 93.98))
+    (stroke (width 0) (type default))
+  )
   (wire (pts (xy 154.94 50.8) (xy 157.48 50.8))
     (stroke (width 0) (type default))
@@
     (stroke (width 0) (type default))
   )
+  (wire (pts (xy 167.64 82.55) (xy 190.5 82.55))
+    (stroke (width 0) (type default))
+  )
   (wire (pts (xy 170.18 87.63) (xy 167.64 87.63))
     (stroke (width 0) (type default))
@@
     (stroke (width 0) (type default))
   )
-  (wire (pts (xy 129.54 67.31) (xy 137.16 67.31))
+  (wire (pts (xy 101.6 67.31) (xy 137.16 67.31))
     (stroke (width 0) (type default))
   )
@@
     (stroke (width 0) (type default))
   )
-  (wire (pts (xy 149.86 45.72) (xy 149.86 50.8))
+  (wire (pts (xy 114.3 54.61) (xy 114.3 62.23))
+    (stroke (width 0) (type default))
+  )
+  (wire (pts (xy 149.86 35.56) (xy 149.86 50.8))
     (stroke (width 0) (type default))
   )
@@
     (stroke (width 0) (type default))
   )
-  (wire (pts (xy 154.94 45.72) (xy 154.94 50.8))
+  (wire (pts (xy 154.94 35.56) (xy 154.94 36.83))
     (stroke (width 0) (type default))
   )
@@
     (stroke (width 0) (type default))
   )
-  (wire (pts (xy 170.18 90.17) (xy 177.8 90.17))
-    (stroke (width 0) (type default))
-  )
-  (wire (pts (xy 129.54 72.39) (xy 137.16 72.39))
+  (wire (pts (xy 190.5 91.44) (xy 190.5 93.98))
+    (stroke (width 0) (type default))
+  )
+  (wire (pts (xy 101.6 72.39) (xy 137.16 72.39))
     (stroke (width 0) (type default))
   )
@@
     (stroke (width 0) (type default))
   )
-  (wire (pts (xy 167.64 82.55) (xy 177.8 82.55))
-    (stroke (width 0) (type default))
-  )
-  (wire (pts (xy 129.54 69.85) (xy 137.16 69.85))
+  (wire (pts (xy 114.3 62.23) (xy 137.16 62.23))
+    (stroke (width 0) (type default))
+  )
+  (wire (pts (xy 101.6 69.85) (xy 137.16 69.85))
     (stroke (width 0) (type default))
   )
@@
     (stroke (width 0) (type default))
   )
+  (wire (pts (xy 101.6 62.23) (xy 114.3 62.23))
+    (stroke (width 0) (type default))
+  )
   (wire (pts (xy 170.18 77.47) (xy 170.18 80.01))
     (stroke (width 0) (type default))
@@
     (stroke (width 0) (type default))
   )
+  (wire (pts (xy 190.5 82.55) (xy 217.17 82.55))
+    (stroke (width 0) (type default))
+  )
   (wire (pts (xy 177.8 72.39) (xy 170.18 72.39))
     (stroke (width 0) (type default))
   )
-  (wire (pts (xy 170.18 77.47) (xy 177.8 77.47))
+  (wire (pts (xy 170.18 77.47) (xy 217.17 77.47))
+    (stroke (width 0) (type default))
+  )
+  (wire (pts (xy 154.94 41.91) (xy 154.94 50.8))
     (stroke (width 0) (type default))
   )
   (wire (pts (xy 167.64 62.23) (xy 170.18 62.23))
+    (stroke (width 0) (type default))
+  )
+  (wire (pts (xy 170.18 90.17) (xy 170.18 93.98))
+    (stroke (width 0) (type default))
+  )
+  (wire (pts (xy 190.5 93.98) (xy 217.17 93.98))
     (stroke (width 0) (type default))
   )
@@
     (effects (font (size 1.27 1.27)) (justify left bottom))
   )
-  (hierarchical_label "~{CS}" (shape input) (at 129.54 69.85 180) (fields_autoplaced)
-    (effects (font (size 1.27 1.27)) (justify right))
-  )
-  (hierarchical_label "MOSI" (shape input) (at 129.54 64.77 180) (fields_autoplaced)
-    (effects (font (size 1.27 1.27)) (justify right))
-  )
-  (hierarchical_label "SCLK" (shape input) (at 129.54 67.31 180) (fields_autoplaced)
+  (hierarchical_label "~{DATA_READY}" (shape output) (at 101.6 62.23 180) (fields_autoplaced)
+    (effects (font (size 1.27 1.27)) (justify right))
+  )
+  (hierarchical_label "~{CS}" (shape input) (at 101.6 69.85 180) (fields_autoplaced)
+    (effects (font (size 1.27 1.27)) (justify right))
+  )
+  (hierarchical_label "PT100_-IN" (shape input) (at 217.17 93.98 0) (fields_autoplaced)
+    (effects (font (size 1.27 1.27)) (justify left))
+  )
+  (hierarchical_label "PT100_+IN" (shape input) (at 217.17 82.55 0) (fields_autoplaced)
+    (effects (font (size 1.27 1.27)) (justify left))
+  )
+  (hierarchical_label "MOSI" (shape input) (at 101.6 64.77 180) (fields_autoplaced)
+    (effects (font (size 1.27 1.27)) (justify right))
+  )
+  (hierarchical_label "PT100_+OUT" (shape output) (at 217.17 77.47 0) (fields_autoplaced)
+    (effects (font (size 1.27 1.27)) (justify left))
+  )
+  (hierarchical_label "SCLK" (shape input) (at 101.6 67.31 180) (fields_autoplaced)
     (effects (font (size 1.27 1.27)) (justify right))
   )
@@
     (effects (font (size 1.27 1.27)) (justify right))
   )
-  (hierarchical_label "+3.3VD" (shape input) (at 154.94 45.72 90) (fields_autoplaced)
-    (effects (font (size 1.27 1.27)) (justify left))
-  )
-  (hierarchical_label "MISO" (shape output) (at 129.54 72.39 180) (fields_autoplaced)
+  (hierarchical_label "+3.3VD" (shape input) (at 154.94 35.56 90) (fields_autoplaced)
+    (effects (font (size 1.27 1.27)) (justify left))
+  )
+  (hierarchical_label "MISO" (shape output) (at 101.6 72.39 180) (fields_autoplaced)
     (effects (font (size 1.27 1.27)) (justify right))
   )
@@
     (effects (font (size 1.27 1.27)) (justify right))
   )
-  (hierarchical_label "+3.3VD" (shape input) (at 149.86 45.72 90) (fields_autoplaced)
+  (hierarchical_label "+3.3VD" (shape input) (at 149.86 35.56 90) (fields_autoplaced)
     (effects (font (size 1.27 1.27)) (justify left))
   )
@@
     )
   )
+  (symbol (lib_id "Device:C") (at 190.5 87.63 180) (unit 1)
+    (in_bom yes) (on_board yes) (dnp no) (fields_autoplaced)
+    (property "Reference" "C3" (at 194.31 86.995 0)
+      (effects (font (size 1.27 1.27)) (justify right))
+    )
+    (property "Value" "10n" (at 194.31 89.535 0)
+      (effects (font (size 1.27 1.27)) (justify right))
+    )
+    (property "Footprint" "Capacitor_SMD:C_1206_3216Metric" (at 189.5348 83.82 0)
+      (effects (font (size 1.27 1.27)) hide)
+    )
+    (property "Datasheet" "~" (at 190.5 87.63 0)
+      (effects (font (size 1.27 1.27)) hide)
+    )
+    (pin "1")
+    (pin "2")
+    (instances
+      (project "ReflowController"
+        (path "/2394cc2a-b9b0-4c0b-be11-1fc6085b0d5c/cedd135a-27b6-4ce6-9f5e-bdcd93291ccf"
+          (reference "C3") (unit 1)
+        )
+      )
+    )
+  )
   (symbol (lib_id "Device:C") (at 143.51 50.8 270) (unit 1)
     (in_bom yes) (on_board yes) (dnp no) (fields_autoplaced)
@@
       (effects (font (size 1.27 1.27)) (justify left))
     )
-    (property "Value" "R" (at 180.34 69.215 0)
+    (property "Value" "402" (at 180.34 69.215 0)
       (effects (font (size 1.27 1.27)) (justify left))
     )
@@
         )
       )
+    )
+  )
+  (symbol (lib_id "Connector:TestPoint") (at 114.3 54.61 0) (unit 1)
+    (in_bom yes) (on_board yes) (dnp no) (fields_autoplaced)
+    (property "Reference" "TP1" (at 116.84 50.673 0)
+      (effects (font (size 1.27 1.27)) (justify left))
+    )
+    (property "Value" "T_RDY" (at 116.84 53.213 0)
+      (effects (font (size 1.27 1.27)) (justify left))
+    )
+    (property "Footprint" "" (at 119.38 54.61 0)
+      (effects (font (size 1.27 1.27)) hide)
+    )
+    (property "Datasheet" "~" (at 119.38 54.61 0)
+      (effects (font (size 1.27 1.27)) hide)
+    )
+    (pin "1")
+    (instances
+      (project "ReflowController"
+        (path "/2394cc2a-b9b0-4c0b-be11-1fc6085b0d5c/cedd135a-27b6-4ce6-9f5e-bdcd93291ccf"
+          (reference "TP1") (unit 1)
+        )
+      )
+    )
+  )
+  (symbol (lib_id "Device:NetTie_2") (at 154.94 39.37 90) (unit 1)
+    (in_bom no) (on_board yes) (dnp no) (fields_autoplaced)
+    (property "Reference" "NT3" (at 156.21 38.735 90)
+      (effects (font (size 1.27 1.27)) (justify right))
+    )
+    (property "Value" "NetTie_2" (at 156.21 41.275 90)
+      (effects (font (size 1.27 1.27)) (justify right))
+    )
+    (property "Footprint" "" (at 154.94 39.37 0)
+      (effects (font (size 1.27 1.27)) hide)
+    )
+    (property "Datasheet" "~" (at 154.94 39.37 0)
+      (effects (font (size 1.27 1.27)) hide)
+    )
+    (pin "1")
+    (pin "2")
+    (instances
+      (project "ReflowController"
+        (path "/2394cc2a-b9b0-4c0b-be11-1fc6085b0d5c/cedd135a-27b6-4ce6-9f5e-bdcd93291ccf"
+          (reference "NT3") (unit 1)
+        )
+      )

Commit message: work on MAX31865 circuit
Parts:
- removed TP1: T_RDY, symbol Connector:TestPoint
- added D1, D2, D3: SMLVT3V3, symbol Device:D_Zener
- added R2: 10M, Resistor_SMD:R_1206_3216Metric, symbol Device:R
- added R3: 10k, Resistor_SMD:R_1206_3216Metric, symbol Device:R
- C1, C2, C3: type (none) -> NP0/C0G
- R1: TC (none) -> 10ppm; manNo (none) -> RQ73C2B402RBTD; pow (none) -> 0.4W; tol (none) -> 0.1%
Connections:
- net +3.3VD: now also R3.1
- net PT100_+IN: now also D1.1 (K), R2.2
- net PT100_+OUT: now also D3.1 (K)
- net PT100_-IN: now also D2.1 (K)
- net ~{CS}: now also R3.2
- net at NT3.1, U4.3 (VDD): now also C2.2; no longer C2.1
- net REFIN+: now reaches R1.1, U4.4 (BIAS), U4.5 (REFIN+)
- net REFIN+: now also R2.1
- net REFIN-: now reaches R1.2, U4.6 (REFIN-), U4.7 (ISENSOR)
- net AGND renamed T_AGND
- net T_AGND: now also C2.1, D1.2 (A), D2.2 (A), D3.2 (A); no longer C2.2
Other:
- note removed: "TODO: - add protection diodes to all 4x wires - make a circuit with dipswitches to infrom system if 4x wire or 3x wire sense is used - figure out circuit to switch between PT100 and PT1000"
- moved on the sheet: C1, C3, NT2, NT3, R1, U4
