File: Hardware/ReflowController/ReflowController.kicad_sch (KiCad schematic)
At the start: 3 parts

Commit message: started with schematic
Other:
- sheet TemperatureReader ports: added +3.3VD, ~{CS}; removed +5VD, CS

Commit message: work on temp ic circuit
Other:
- sheet TemperatureReader ports: added PT100_+IN, PT100_+OUT, PT100_-IN, ~{DATA_READY}; removed none
Changed lines of the file:
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@@
     )
   )
-  (sheet (at 199.39 46.99) (size 22.86 29.21) (fields_autoplaced)
+  (sheet (at 199.39 46.99) (size 29.21 29.21) (fields_autoplaced)
     (stroke (width 0.1524) (type solid))
     (fill (color 0 0 0 0.0000))
@@
       (effects (font (size 1.27 1.27)) (justify left))
     )
+    (pin "PT100_+IN" input (at 228.6 57.15 0)
+      (effects (font (size 1.27 1.27)) (justify right))
+    )
+    (pin "PT100_+OUT" output (at 228.6 59.69 0)
+      (effects (font (size 1.27 1.27)) (justify right))
+    )
+    (pin "PT100_-IN" input (at 228.6 62.23 0)
+      (effects (font (size 1.27 1.27)) (justify right))
+    )
+    (pin "~{DATA_READY}" output (at 199.39 60.96 180)
+      (effects (font (size 1.27 1.27)) (justify left))
+    )

Commit message: work on schematic
Parts:
- added J1: Conn_01x03_Socket, symbol Connector:Conn_01x03_Socket
Connections:
- net TemperatureReader/PT100_+IN: now also J1.1 (Pin_1)
- net TemperatureReader/PT100_+OUT: now also J1.2 (Pin_2)
- net TemperatureReader/PT100_-IN: now also J1.3 (Pin_3)
Other:
- note added: "TODO: - Find out what connector"
Changed lines of the file:
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@@
+    (stroke (width 0) (type default))
+  )
+  (wire (pts (xy 195.58 50.8) (xy 195.58 48.26))
     (stroke (width 0) (type default))
   )
@@
     (stroke (width 0) (type default))
   )
+  (wire (pts (xy 228.6 50.8) (xy 241.3 50.8))
+    (stroke (width 0) (type default))
+  )
   (wire (pts (xy 96.52 63.5) (xy 113.03 63.5))
     (stroke (width 0) (type default))
@@
     (stroke (width 0) (type default))
   )
+  (wire (pts (xy 199.39 54.61) (xy 195.58 54.61))
+    (stroke (width 0) (type default))
+  )
   (wire (pts (xy 121.92 53.34) (xy 127 53.34))
     (stroke (width 0) (type default))
@@
     (stroke (width 0) (type default))
   )
+  (wire (pts (xy 228.6 55.88) (xy 241.3 55.88))
+    (stroke (width 0) (type default))
+  )
   (wire (pts (xy 121.92 50.8) (xy 121.92 49.53))
     (stroke (width 0) (type default))
@@
     (stroke (width 0) (type default))
   )
+  (wire (pts (xy 195.58 54.61) (xy 195.58 57.15))
+    (stroke (width 0) (type default))
+  )
   (wire (pts (xy 121.92 54.61) (xy 121.92 53.34))
     (stroke (width 0) (type default))
@@
     (stroke (width 0) (type default))
   )
+  (wire (pts (xy 199.39 50.8) (xy 195.58 50.8))
+    (stroke (width 0) (type default))
+  )
   (wire (pts (xy 127 50.8) (xy 121.92 50.8))
+    (stroke (width 0) (type default))
+  )
+  (wire (pts (xy 228.6 53.34) (xy 241.3 53.34))
     (stroke (width 0) (type default))
   )
@@
     (effects (font (size 1.27 1.27)) (justify left bottom))
   )
+  (text "TODO:\n- Find out what connector\n" (at 248.92 53.34 0)
+    (effects (font (size 1.27 1.27)) (justify left bottom))
+  )
   (label "COM" (at 144.78 17.78 0) (fields_autoplaced)
     (effects (font (size 1.27 1.27)) (justify left bottom))
@@
     (effects (font (size 1.27 1.27)) (justify left bottom))
   )
-  (label "CS_TEMP" (at 180.34 71.12 0) (fields_autoplaced)
-    (effects (font (size 1.27 1.27)) (justify left bottom))
+  (label "~{CS_TEMP}" (at 180.34 71.12 0) (fields_autoplaced)
+    (effects (font (size 1.27 1.27)) (justify left bottom))
+  )
+  (symbol (lib_id "power:+3.3V") (at 195.58 48.26 0) (unit 1)
+    (in_bom yes) (on_board yes) (dnp no) (fields_autoplaced)
+    (property "Reference" "#PWR09" (at 195.58 52.07 0)
+      (effects (font (size 1.27 1.27)) hide)
+    )
+    (property "Value" "+3.3V" (at 195.58 44.45 0)
+      (effects (font (size 1.27 1.27)))
+    )
+    (property "Footprint" "" (at 195.58 48.26 0)
+      (effects (font (size 1.27 1.27)) hide)
+    )
+    (property "Datasheet" "" (at 195.58 48.26 0)
+      (effects (font (size 1.27 1.27)) hide)
+    )
+    (pin "1")
+    (instances
+      (project "ReflowController"
+        (path "/2394cc2a-b9b0-4c0b-be11-1fc6085b0d5c"
+          (reference "#PWR09") (unit 1)
+        )
+      )
+    )
   )
   (symbol (lib_id "Device:R") (at 123.19 120.65 90) (unit 1)
@@
     )
   )
+  (symbol (lib_id "power:GNDD") (at 195.58 57.15 0) (unit 1)
+    (in_bom yes) (on_board yes) (dnp no)
+    (property "Reference" "#PWR08" (at 195.58 63.5 0)
+      (effects (font (size 1.27 1.27)) hide)
+    )
+    (property "Value" "GNDD" (at 195.58 60.96 0)
+      (effects (font (size 1.27 1.27)))
+    )
+    (property "Footprint" "" (at 195.58 57.15 0)
+      (effects (font (size 1.27 1.27)) hide)
+    )
+    (property "Datasheet" "" (at 195.58 57.15 0)
+      (effects (font (size 1.27 1.27)) hide)
+    )
+    (pin "1")
+    (instances
+      (project "ReflowController"
+        (path "/2394cc2a-b9b0-4c0b-be11-1fc6085b0d5c"
+          (reference "#PWR08") (unit 1)
+        )
+      )
+    )
+  )
   (symbol (lib_id "power:+5VD") (at 121.92 49.53 0) (unit 1)
     (in_bom yes) (on_board yes) (dnp no) (fields_autoplaced)
@@
         (path "/2394cc2a-b9b0-4c0b-be11-1fc6085b0d5c"
           (reference "#PWR07") (unit 1)
+        )
+      )
+    )
+  )
+  (symbol (lib_id "Connector:Conn_01x03_Socket") (at 246.38 53.34 0) (unit 1)
+    (in_bom yes) (on_board yes) (dnp no)
+    (property "Reference" "J1" (at 241.3 44.45 0)
+      (effects (font (size 1.27 1.27)) (justify left))
+    )
+    (property "Value" "Conn_01x03_Socket" (at 241.3 46.99 0)
+      (effects (font (size 1.27 1.27)) (justify left))
+    )
+    (property "Footprint" "" (at 246.38 53.34 0)
+      (effects (font (size 1.27 1.27)) hide)
+    )
+    (property "Datasheet" "~" (at 246.38 53.34 0)
+      (effects (font (size 1.27 1.27)) hide)
+    )
+    (pin "1")
+    (pin "2")
+    (pin "3")
+    (instances
+      (project "ReflowController"
+        (path "/2394cc2a-b9b0-4c0b-be11-1fc6085b0d5c"
+          (reference "J1") (unit 1)
         )
       )
@@
       (effects (font (size 1.27 1.27)) (justify left))
     )
-    (pin "PT100_+IN" input (at 228.6 57.15 0)
-      (effects (font (size 1.27 1.27)) (justify right))
-    )
-    (pin "PT100_+OUT" output (at 228.6 59.69 0)
-      (effects (font (size 1.27 1.27)) (justify right))
-    )
-    (pin "PT100_-IN" input (at 228.6 62.23 0)
-      (effects (font (size 1.27 1.27)) (justify right))
-    )
+    (pin "PT100_+IN" input (at 228.6 50.8 0)
+      (effects (font (size 1.27 1.27)) (justify right))
+    )
+    (pin "PT100_+OUT" output (at 228.6 53.34 0)
+      (effects (font (size 1.27 1.27)) (justify right))
+    )
+    (pin "PT100_-IN" input (at 228.6 55.88 0)
+      (effects (font (size 1.27 1.27)) (justify right))
+    )

Commit message: work on circuit
Other:
- note removed: "TODO: - Find out what connector"
- moved on the sheet: J1
Changed lines of the file:
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@@
     (stroke (width 0) (type default))
   )
-  (wire (pts (xy 180.34 63.5) (xy 199.39 63.5))
-    (stroke (width 0) (type default))
-  )
-  (wire (pts (xy 195.58 50.8) (xy 195.58 48.26))
+  (wire (pts (xy 180.34 63.5) (xy 203.2 63.5))
+    (stroke (width 0) (type default))
+  )
+  (wire (pts (xy 199.39 50.8) (xy 199.39 48.26))
     (stroke (width 0) (type default))
   )
@@
     (stroke (width 0) (type default))
   )
-  (wire (pts (xy 228.6 50.8) (xy 241.3 50.8))
+  (wire (pts (xy 228.6 50.8) (xy 240.03 50.8))
     (stroke (width 0) (type default))
   )
@@
     (stroke (width 0) (type default))
   )
-  (wire (pts (xy 199.39 54.61) (xy 195.58 54.61))
+  (wire (pts (xy 203.2 54.61) (xy 199.39 54.61))
     (stroke (width 0) (type default))
   )
@@
     (stroke (width 0) (type default))
   )
-  (wire (pts (xy 228.6 55.88) (xy 241.3 55.88))
+  (wire (pts (xy 228.6 55.88) (xy 240.03 55.88))
     (stroke (width 0) (type default))
   )
@@
     (stroke (width 0) (type default))
   )
-  (wire (pts (xy 180.34 68.58) (xy 199.39 68.58))
-    (stroke (width 0) (type default))
-  )
-  (wire (pts (xy 180.34 66.04) (xy 199.39 66.04))
-    (stroke (width 0) (type default))
-  )
-  (wire (pts (xy 180.34 71.12) (xy 199.39 71.12))
+  (wire (pts (xy 180.34 66.04) (xy 203.2 66.04))
+    (stroke (width 0) (type default))
+  )
+  (wire (pts (xy 180.34 71.12) (xy 203.2 71.12))
     (stroke (width 0) (type default))
   )
@@
     (stroke (width 0) (type default))
   )
-  (wire (pts (xy 195.58 54.61) (xy 195.58 57.15))
+  (wire (pts (xy 199.39 54.61) (xy 199.39 57.15))
     (stroke (width 0) (type default))
   )
@@
     (stroke (width 0) (type default))
   )
-  (wire (pts (xy 199.39 50.8) (xy 195.58 50.8))
+  (wire (pts (xy 203.2 50.8) (xy 199.39 50.8))
     (stroke (width 0) (type default))
   )
@@
     (stroke (width 0) (type default))
   )
-  (wire (pts (xy 228.6 53.34) (xy 241.3 53.34))
+  (wire (pts (xy 228.6 53.34) (xy 240.03 53.34))
     (stroke (width 0) (type default))
   )
@@
   )
   (bus (pts (xy 177.8 17.78) (xy 177.8 60.96))
+    (stroke (width 0) (type default))
+  )
+  (wire (pts (xy 180.34 68.58) (xy 203.2 68.58))
     (stroke (width 0) (type default))
   )
@@
     (effects (font (size 1.27 1.27)) (justify left bottom))
   )
-  (text "TODO:\n- Find out what connector\n" (at 248.92 53.34 0)
-    (effects (font (size 1.27 1.27)) (justify left bottom))
-  )
   (label "COM" (at 144.78 17.78 0) (fields_autoplaced)
     (effects (font (size 1.27 1.27)) (justify left bottom))
@@
     (effects (font (size 1.27 1.27)) (justify left bottom))
   )
-  (symbol (lib_id "power:+3.3V") (at 195.58 48.26 0) (unit 1)
-    (in_bom yes) (on_board yes) (dnp no) (fields_autoplaced)
-    (property "Reference" "#PWR09" (at 195.58 52.07 0)
-      (effects (font (size 1.27 1.27)) hide)
-    )
-    (property "Value" "+3.3V" (at 195.58 44.45 0)
-      (effects (font (size 1.27 1.27)))
-    )
-    (property "Footprint" "" (at 195.58 48.26 0)
-      (effects (font (size 1.27 1.27)) hide)
-    )
-    (property "Datasheet" "" (at 195.58 48.26 0)
+  (symbol (lib_id "power:+3.3V") (at 199.39 48.26 0) (unit 1)
+    (in_bom yes) (on_board yes) (dnp no) (fields_autoplaced)
+    (property "Reference" "#PWR09" (at 199.39 52.07 0)
+      (effects (font (size 1.27 1.27)) hide)
+    )
+    (property "Value" "+3.3V" (at 199.39 44.45 0)
+      (effects (font (size 1.27 1.27)))
+    )
+    (property "Footprint" "" (at 199.39 48.26 0)
+      (effects (font (size 1.27 1.27)) hide)
+    )
+    (property "Datasheet" "" (at 199.39 48.26 0)
       (effects (font (size 1.27 1.27)) hide)
     )
@@
     )
   )
-  (symbol (lib_id "power:GNDD") (at 195.58 57.15 0) (unit 1)
+  (symbol (lib_id "power:GNDD") (at 199.39 57.15 0) (unit 1)
     (in_bom yes) (on_board yes) (dnp no)
-    (property "Reference" "#PWR08" (at 195.58 63.5 0)
-      (effects (font (size 1.27 1.27)) hide)
-    )
-    (property "Value" "GNDD" (at 195.58 60.96 0)
-      (effects (font (size 1.27 1.27)))
-    )
-    (property "Footprint" "" (at 195.58 57.15 0)
-      (effects (font (size 1.27 1.27)) hide)
-    )
-    (property "Datasheet" "" (at 195.58 57.15 0)
+    (property "Reference" "#PWR08" (at 199.39 63.5 0)
+      (effects (font (size 1.27 1.27)) hide)
+    )
+    (property "Value" "GNDD" (at 199.39 60.96 0)
+      (effects (font (size 1.27 1.27)))
+    )
+    (property "Footprint" "" (at 199.39 57.15 0)
+      (effects (font (size 1.27 1.27)) hide)
+    )
+    (property "Datasheet" "" (at 199.39 57.15 0)
       (effects (font (size 1.27 1.27)) hide)
     )
@@
     )
   )
-  (symbol (lib_id "Connector:Conn_01x03_Socket") (at 246.38 53.34 0) (unit 1)
+  (symbol (lib_id "Connector:Conn_01x03_Socket") (at 245.11 53.34 0) (unit 1)
     (in_bom yes) (on_board yes) (dnp no)
-    (property "Reference" "J1" (at 241.3 44.45 0)
-      (effects (font (size 1.27 1.27)) (justify left))
-    )
-    (property "Value" "Conn_01x03_Socket" (at 241.3 46.99 0)
-      (effects (font (size 1.27 1.27)) (justify left))
-    )
-    (property "Footprint" "" (at 246.38 53.34 0)
-      (effects (font (size 1.27 1.27)) hide)
-    )
-    (property "Datasheet" "~" (at 246.38 53.34 0)
+    (property "Reference" "J1" (at 240.03 44.45 0)
+      (effects (font (size 1.27 1.27)) (justify left))
+    )
+    (property "Value" "Conn_01x03_Socket" (at 240.03 46.99 0)
+      (effects (font (size 1.27 1.27)) (justify left))
+    )
+    (property "Footprint" "" (at 245.11 53.34 0)
+      (effects (font (size 1.27 1.27)) hide)
+    )
+    (property "Datasheet" "~" (at 245.11 53.34 0)
       (effects (font (size 1.27 1.27)) hide)
     )
@@
     )
   )
-  (sheet (at 199.39 46.99) (size 29.21 29.21) (fields_autoplaced)
+  (sheet (at 203.2 46.99) (size 25.4 29.21) (fields_autoplaced)
     (stroke (width 0.1524) (type solid))
     (fill (color 0 0 0 0.0000))
-    (property "Sheetname" "TemperatureReader" (at 199.39 46.2784 0)
+    (property "Sheetname" "TemperatureReader" (at 203.2 46.2784 0)
       (effects (font (size 1.27 1.27)) (justify left bottom))
     )
-    (property "Sheetfile" "TemperatureReader.kicad_sch" (at 199.39 76.7846 0)
+    (property "Sheetfile" "TemperatureReader.kicad_sch" (at 203.2 76.7846 0)
       (effects (font (size 1.27 1.27)) (justify left top))
     )
-    (pin "DGND" passive (at 199.39 54.61 180)
-      (effects (font (size 1.27 1.27)) (justify left))
-    )
-    (pin "+3.3VD" input (at 199.39 50.8 180)
-      (effects (font (size 1.27 1.27)) (justify left))
-    )
-    (pin "MOSI" input (at 199.39 63.5 180)
-      (effects (font (size 1.27 1.27)) (justify left))
-    )
-    (pin "SCLK" input (at 199.39 68.58 180)
-      (effects (font (size 1.27 1.27)) (justify left))
-    )
-    (pin "MISO" output (at 199.39 66.04 180)
-      (effects (font (size 1.27 1.27)) (justify left))
-    )
-    (pin "~{CS}" input (at 199.39 71.12 180)
+    (pin "DGND" passive (at 203.2 54.61 180)
+      (effects (font (size 1.27 1.27)) (justify left))
+    )
+    (pin "+3.3VD" input (at 203.2 50.8 180)
+      (effects (font (size 1.27 1.27)) (justify left))
+    )
+    (pin "MOSI" input (at 203.2 63.5 180)
+      (effects (font (size 1.27 1.27)) (justify left))
+    )
+    (pin "SCLK" input (at 203.2 68.58 180)
+      (effects (font (size 1.27 1.27)) (justify left))
+    )
+    (pin "MISO" output (at 203.2 66.04 180)
+      (effects (font (size 1.27 1.27)) (justify left))
+    )
+    (pin "~{CS}" input (at 203.2 71.12 180)
       (effects (font (size 1.27 1.27)) (justify left))
     )
@@
       (effects (font (size 1.27 1.27)) (justify right))
     )
-    (pin "~{DATA_READY}" output (at 199.39 60.96 180)
-      (effects (font (size 1.27 1.27)) (justify left))
-    )
+    (pin "~{DATA_READY}" output (at 203.2 60.96 180)
+      (effects (font (size 1.27 1.27)) (justify left))
+    )
