File: Hardware/ReflowController/uC.kicad_sch (KiCad schematic)
At the start: 33 parts, among them J1 Conn_01x15_Female, J2 Conn_01x15_Female

Commit message: work on uC schematic
Parts:
- removed J1, J2: Conn_01x15_Female, symbol Connector:Conn_01x15_Female
- removed NT10, NT11, NT12, NT13, NT14, NT15, NT16, NT17, NT18, NT19, NT2, NT20, NT21, NT22, NT23, NT24, NT25, NT26, NT27, NT28, NT29, NT3, NT30, NT31, NT8, NT9: NetTie_2, symbol Device:NetTie_2
- added A1: NUCLEO_STM32F042K6, Module:Arduino_Nano, symbol MCU_Module:Arduino_Nano_v3.x
- added R2 (x2): 4k7, Resistor_SMD:R_1206_3216Metric, symbol Device:R
Connections:
- net +5VD: now also A1.27 (+5V)
- net AREF: now also A1.18 (AREF)
- net DGND: now also A1.29 (GND), A1.4 (GND)
- net MISO: now also NT4.2
- net MOSI: now also NT1.2
- net PA0: now also A1.19 (A0)
- net PA1: now also A1.20 (A1)
- net PA10: now also A1.1 (D1/TX)
- net PA11: now also A1.13 (D10)
- net PA12: now also A1.5 (D2)
- net PA2: now also A1.26 (A7)
- net PA3: now also A1.21 (A2)
- net PA4: now also NT5.1, A1.22 (A3); no longer NT1.1
- net PA5: now also A1.23 (A4)
- net PA6: now also NT4.1, A1.24 (A5)
- net PA7: now also NT1.1, A1.25 (A6)
- net PA8: now also A1.12 (D9)
- net PA9: now also A1.2 (D0/RX)
- net PB0: now also A1.6 (D3)
- net PB1: now also A1.9 (D6)
- net PB3: now also A1.16 (D13)
- net PB4: now also A1.15 (D12)
- net PB5: now also A1.14 (D11)
- net PB6: now also NT7.1, A1.8 (D5)
- net PB7: now also NT6.1, A1.7 (D4)
- net PF0: now also A1.10 (D7)
- net PF1: now also A1.11 (D8)
- net SCL: now also NT7.2, R2.2
- net SCLK: now also NT5.2; no longer NT1.2
- net SDA: now also NT6.2, R2.2
- new net +3.3VD: R2.1, R2.1
- new net ~{RESET}: A1.28 (~{RESET})
Other:
- note added: "I2C"
- note added: "NOTES"
- note added: "SPI"
- note added: "[1]"
- note added: "[1] : Please refer to the user manual UM1956 for further schematic information regarding the NUCLEO board"
- note added: "[2]"
- note added: "[2] : External 5V can be fed in while ST-Link also feeds the NUCLEO. The needed 3.3VD are generated on board from the 5VD."
