File: Hardware/ReflowController/ReflowController.kicad_pcb (KiCad board)
At the start: 4 copper layers, 160 x 100 mm, 152 parts, among them J101 2060-1452, J102 2060-1452, J103 2060-1453, J104 2060-1452, J105 2060-1452, J106 2060-1452, J107 2060-1452, J108 2060-1452, J109 2060-1452, J110 2060-1452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

Commit message: work on the layout
Parts:
- moved R710 23.8 mm to (170.0, 119.5)
- moved R709 21.4 mm to (172.5, 116.5), turned to 180 degrees
- moved R708 12.9 mm to (181.0, 119.0)
- moved R707 10.2 mm to (185.0, 120.5), turned to 180 degrees
- moved C702 1.75 mm to (183.2, 109.5)
- moved D701 0.75 mm to (186.0, 107.0)
- moved R706 0.75 mm to (189.2, 108.5)
Routing:
- net +24V: track 172.4 -> 204.7 mm, vias 22 -> 24
- net Net-(D701-A): track 0.00 -> 14.7 mm
- net /IO/HSS_4_OUT_+: track 19.4 -> 33.0 mm
- net /IO/HSS_1_OUT_+: track 16.9 -> 28.9 mm
- net /IO/HSS_3_OUT_+: track 14.8 -> 26.1 mm
- net /IO/HSS_2_OUT_+: track 13.1 -> 24.4 mm
- net GNDPWR: vias 49 -> 53
- added copper zone on B.Cu, net Earth
- added copper zone on In2.Cu, net Earth

Commit message: work on layout
Parts:
- moved R501 6.06 mm to (137.7, 107.7), turned to 180 degrees
- moved C505 4.39 mm to (131.8, 105.0)
- moved R503 3.05 mm to (131.8, 107.1), turned to 0 degrees
- moved C501 2.27 mm to (130.0, 108.6), turned to 180 degrees
- moved NT6 1.00 mm to (91.6, 98.5)
- moved NT14 0.42 mm to (94.1, 98.6)
- moved NT11 0.10 mm to (84.0, 98.5)
- moved NT12 0.10 mm to (96.7, 98.6)
Routing:
- net /uC/~{INT_EMERGENCY_STOP}: track 0.00 -> 94.8 mm, vias 0 -> 1
- net +24V: track 204.7 -> 241.8 mm, vias 24 -> 26
- net GNDPWR: track 95.6 -> 105.3 mm, vias 53 -> 44
- net /Fan Driver/FAN_1_OUT_-: track 9.83 -> 19.0 mm
- net /Fan Driver/FAN_1_OUT_+: track 15.0 -> 23.6 mm
- net /FAN_2_EN: track 5.02 -> 12.2 mm
- net /FAN_2_PWM: track 5.10 -> 12.1 mm, vias 0 -> 1
- net +5V: track 6.67 -> 13.1 mm
- net GND: track 60.9 -> 57.2 mm, vias 50 -> 48
- net /FAN_1_PWM: track 5.31 -> 8.53 mm
- net /uC/PA1: track 0.00 -> 2.05 mm
- net /uC/PA5: track 0.00 -> 2.04 mm
- net /uC/PA7: track 0.00 -> 1.95 mm
- net /uC/PA6: track 0.00 -> 1.94 mm
- net /uC/PA2: track 0.00 -> 1.93 mm
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
Commit message: work on lyout
Routing:
- net /RELAY_1_EN: track 1.66 -> 107.3 mm, vias 0 -> 1
- net +5V: track 13.1 -> 71.6 mm, vias 8 -> 9
- net /FAN_2_PWM: track 12.1 -> 57.0 mm, vias 1 -> 3
- net /FAN_1_PWM: track 8.53 -> 45.6 mm, vias 0 -> 3
- net /FAN_1_EN: track 6.86 -> 41.0 mm, vias 0 -> 2
- net /FAN_2_EN: track 12.2 -> 46.1 mm, vias 0 -> 2
- net +24V: track 241.8 -> 226.5 mm
- net GNDPWR: track 105.3 -> 102.1 mm
- net /uC/~{INT_EMERGENCY_STOP}: track 94.8 -> 96.8 mm
- net /~{UI_RESET}: track 0.00 -> 1.61 mm, vias 0 -> 1
- net /RELAY_2_EN: track 1.61 -> 2.91 mm, vias 0 -> 1
- net /BUZZER_PWM: track 0.00 -> 1.17 mm, vias 0 -> 1
- net /SDA: track 47.1 -> 46.1 mm

Commit message: work on layout
Parts:
- moved C605 6.09 mm to (194.1, 58.3), turned to -90 degrees
- moved R601 5.87 mm to (209.3, 46.4), turned to 90 degrees
- moved R602 5.81 mm to (209.1, 58.3), turned to 90 degrees
- moved C603 4.15 mm to (211.1, 46.4), turned to 90 degrees
- moved C604 3.72 mm to (211.4, 58.2), turned to -90 degrees
- moved R603 2.42 mm to (192.4, 54.0)
Routing:
- net +3.3V: track 270.0 -> 454.5 mm, vias 15 -> 16
- net /ui/ENCODER_B: track 5.17 -> 97.8 mm
- net /ui/ENCODER_A: track 10.8 -> 90.2 mm
- net /ui/ENCODER_SW: track 3.18 -> 50.8 mm
- net /ui/BTN_RESET: track 13.0 -> 58.3 mm
- net /ui/BTN_RIGHT: track 13.0 -> 54.6 mm
- net /ui/BTN_UP: track 13.1 -> 45.9 mm
- net /ui/BTN_SELECT: track 8.49 -> 37.6 mm
- net GND: track 57.6 -> 28.6 mm
- net /ui/BTN_DOWN: track 10.5 -> 37.5 mm
- net /ui/LED_ERROR: track 0.00 -> 18.8 mm
- net /ui/LED_ALIVE: track 0.00 -> 17.9 mm
- net /uC/~{INT_EMERGENCY_STOP}: track 96.8 -> 101.7 mm, vias 1 -> 2

Commit message: work on laout
Parts:
- moved C702 0.80 mm to (183.2, 108.7)
Routing:
- net /SCL: track 47.3 -> 2.88 mm, vias 0 -> 1
- net /SDA: track 46.1 -> 3.38 mm, vias 0 -> 1
- net /ui/BTN_RET: track 13.5 -> 40.2 mm
- net /ui/BTN_LEFT: track 13.1 -> 33.3 mm, vias 0 -> 2
- net /HSS_3_EN: track 0.00 -> 19.1 mm, vias 0 -> 1
- net /HSS_1_EN: track 0.29 -> 18.1 mm, vias 0 -> 1
- net /HSS_2_EN: track 0.34 -> 17.2 mm, vias 0 -> 1
- net /ui/ENCODER_B: track 97.8 -> 99.3 mm
- net +3.3V: track 454.5 -> 453.4 mm
- net GND: vias 48 -> 49

Commit message: work on layout
Parts:
- added R1: 4.7K, Resistor_SMD:R_0603_1608Metric_Pad0.98x0.95mm_HandSolder, F.Cu at (162.1, 84.2)
- added R2: 4.7K, Resistor_SMD:R_0603_1608Metric_Pad0.98x0.95mm_HandSolder, F.Cu at (162.1, 86.2)
Routing:
- net /RELAY_2_EN: track 2.91 -> 158.2 mm, vias 1 -> 3
- net /~{UI_RESET}: track 1.61 -> 81.5 mm, vias 1 -> 2
- net +24V: track 226.5 -> 275.9 mm, vias 26 -> 27
- net /RELAY_1_EN: track 107.3 -> 152.2 mm, vias 1 -> 3
- net /IO/relay_1_coil_-: track 13.2 -> 23.4 mm
- net +3.3V: track 453.4 -> 463.2 mm
- net /IO/relay_2_coil_-: track 8.20 -> 17.7 mm
- net /IO/relay_2_coil_+: track 13.5 -> 22.6 mm
- net /IO/relay_1_coil_+: track 26.9 -> 34.1 mm
- net /uC/PA12: track 0.00 -> 2.39 mm
- net /uC/PB0: track 0.00 -> 2.37 mm
- net /uC/PA11: track 0.00 -> 2.16 mm
- net /uC/PA8: track 0.00 -> 2.12 mm
- net /SCL: track 2.88 -> 4.54 mm
- net /SDA: track 3.38 -> 4.99 mm

Commit message: working on DRC
Parts:
- moved R23 7.75 mm to (81.5, 82.3), turned to 0 degrees
- moved NT5 3.75 mm to (84.0, 83.9)
- moved R22 2.65 mm to (88.9, 82.3), turned to 180 degrees
Connections:
- H103 pad 1: Earth -> unconnected-(H103-Pad1)
- H104 pad 1: Earth -> unconnected-(H104-Pad1)
Routing:
- net +3.3V: track 463.2 -> 583.7 mm, vias 16 -> 19
- net /~{IO_INT}: track 1.00 -> 100.6 mm, vias 1 -> 3
- net /SCL: track 4.54 -> 103.3 mm, vias 1 -> 3
- net /BUZZER_PWM: track 1.17 -> 98.6 mm, vias 1 -> 3
- net /SDA: track 4.99 -> 101.7 mm, vias 1 -> 3
- net +5V: track 71.6 -> 162.0 mm
- net /HSS_4_EN: track 0.00 -> 13.6 mm, vias 0 -> 1
- net /TemperatureReader/PT100_+OUT: track 30.4 -> 39.6 mm
- net /TemperatureReader/PT100_-IN: track 26.0 -> 35.2 mm
- net /TemperatureReader/PT100_+IN: track 30.0 -> 39.2 mm
- net +24V: track 275.9 -> 267.8 mm
- net /uC/PF1: track 6.96 -> 0.00 mm
- net /FAN_2_PWM: track 57.0 -> 61.5 mm
- net /RELAY_1_EN: track 152.2 -> 155.6 mm
- net /HSS_2_EN: track 17.2 -> 20.0 mm
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- removed copper zone on B.Cu, net +3.3V
