File: Hardware/ReflowController/IO.kicad_sch (KiCad schematic)
At the start: 19 parts, among them U701 VNQ5160K-E, U702 SZNUD3124DMT1G

Commit message: work on BOM cleanup
Parts:
- D14: disit digikey -> (none); disti (none) -> digikey
- R706: Field7 13-RC1206FR-134K7LTR-ND -> (none); disti_no (none) -> 13-RC1206FR-134K7LTR-ND
- U702: dist digikey -> (none); dist_no SZNUD3124DMT1GOSTR-ND -> (none); disti (none) -> digikey; disti_no (none) -> SZNUD3124DMT1GOSTR-ND
Changed lines of the file:
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@@
       (effects (font (size 1.27 1.27)) hide)
     )
-    (property "disit" "digikey" (at 102.235 149.225 90)
+    (property "disit" "" (at 102.235 149.225 90)
       (effects (font (size 1.27 1.27)) hide)
     )
     (property "disti_no" "SBRT5A50SA-13DICT-ND" (at 102.235 149.225 90)
+      (effects (font (size 1.27 1.27)) hide)
+    )
+    (property "disti" "digikey" (at 102.235 149.225 0)
       (effects (font (size 1.27 1.27)) hide)
     )
@@
       (effects (font (size 1.27 1.27)) hide)
     )
-    (property "Field7" "13-RC1206FR-134K7LTR-ND" (at 73.66 99.06 0)
+    (property "Field7" "" (at 73.66 99.06 0)
+      (effects (font (size 1.27 1.27)) hide)
+    )
+    (property "disti_no" "13-RC1206FR-134K7LTR-ND" (at 73.66 99.06 0)
       (effects (font (size 1.27 1.27)) hide)
     )
@@
       (effects (font (size 1.27 1.27)) hide)
     )
-    (property "dist" "digikey" (at 86.36 137.795 0)
-      (effects (font (size 1.27 1.27)) hide)
-    )
-    (property "dist_no" "SZNUD3124DMT1GOSTR-ND" (at 96.52 141.605 0)
+    (property "dist" "" (at 86.36 137.795 0)
+      (effects (font (size 1.27 1.27)) hide)
+    )
+    (property "dist_no" "" (at 96.52 141.605 0)
+      (effects (font (size 1.27 1.27)) hide)
+    )
+    (property "disti" "digikey" (at 78.74 168.275 0)
+      (effects (font (size 1.27 1.27)) hide)
+    )
+    (property "disti_no" "SZNUD3124DMT1GOSTR-ND" (at 78.74 168.275 0)
       (effects (font (size 1.27 1.27)) hide)
     )
@@
       (effects (font (size 1.27 1.27)) hide)
     )
-    (property "disit" "digikey" (at 112.395 149.225 90)
+    (property "disit" "" (at 112.395 149.225 90)
       (effects (font (size 1.27 1.27)) hide)
     )
@@
       (effects (font (size 1.27 1.27)) hide)
     )
+    (property "disti" "digikey" (at 112.395 149.225 0)
+      (effects (font (size 1.27 1.27)) hide)
+    )
