File: Hardware/ReflowController/ui.kicad_sch (KiCad schematic)
At the start: 44 parts, among them J601 LCD_HEADER, Q601 BC848, SW601 RotaryEncoder_Switch, SW602 SW_UP, SW603 SW_DOWN, SW604 SW_LEFT, SW605 SW_RIGHT, SW606 SW_SELECT, SW607 SW_RET, SW608 SW_RESET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

Commit message: work on io adaption
Parts:
- removed D603: BLUE, LED_SMD:LED_0603_1608Metric_Pad1.05x0.95mm_HandSolder, symbol Device:LED
- removed R606: 4.7K, Resistor_SMD:R_0603_1608Metric_Pad0.98x0.95mm_HandSolder, symbol Device:R
Connections:
- net LED_INDICATION: no longer U601.9 (P0_5)
- new net OI_AUX_4: U601.9 (P0_5)
Changed lines of the file:
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@@
   (junction (at 177.165 119.38) (diameter 0) (color 0 0 0 0)
   )
-  (junction (at 119.38 125.095) (diameter 0) (color 0 0 0 0)
-  )
   (junction (at 190.5 52.705) (diameter 0) (color 0 0 0 0)
   )
@@
     (stroke (width 0) (type default))
   )
-  (wire (pts (xy 119.38 125.095) (xy 125.73 125.095))
-    (stroke (width 0) (type default))
-  )
   (wire (pts (xy 190.5 32.385) (xy 190.5 33.655))
     (stroke (width 0) (type default))
   )
-  (wire (pts (xy 125.73 123.19) (xy 125.73 125.095))
-    (stroke (width 0) (type default))
-  )
   (wire (pts (xy 177.8 42.545) (xy 177.8 52.705))
     (stroke (width 0) (type default))
@@
     (stroke (width 0) (type default))
   )
-  (wire (pts (xy 125.73 114.3) (xy 125.73 115.57))
-    (stroke (width 0) (type default))
-  )
   (wire (pts (xy 65.405 128.905) (xy 69.215 128.905))
     (stroke (width 0) (type default))
@@
   )
   (wire (pts (xy 37.465 113.03) (xy 40.64 113.03))
-    (stroke (width 0) (type default))
-  )
-  (wire (pts (xy 125.73 100.965) (xy 125.73 106.68))
     (stroke (width 0) (type default))
   )
@@
     (effects (font (size 1.27 1.27)) (justify right bottom))
   )
-  (label "LED_INDICATION" (at 37.465 145.415 180) (fields_autoplaced)
-    (effects (font (size 1.27 1.27)) (justify right bottom))
-  )
   (label "BTN_RET" (at 67.945 150.495 0) (fields_autoplaced)
     (effects (font (size 1.27 1.27)) (justify left bottom))
@@
     (effects (font (size 1.27 1.27)) (justify right))
   )
+  (hierarchical_label "OI_AUX_4" (shape bidirectional) (at 37.465 145.415 180) (fields_autoplaced)
+    (effects (font (size 1.27 1.27)) (justify right))
+  )
   (hierarchical_label "DGND" (shape passive) (at 108.585 125.095 180) (fields_autoplaced)
     (effects (font (size 1.27 1.27)) (justify right))
@@
         (path "/2394cc2a-b9b0-4c0b-be11-1fc6085b0d5c/c76c60d6-41ab-4683-93d6-43449ec74daf"
           (reference "C601") (unit 1)
-        )
-      )
-    )
-  )
-  (symbol (lib_id "Device:R") (at 125.73 110.49 0) (unit 1)
-    (in_bom yes) (on_board yes) (dnp no)
-    (property "Reference" "R606" (at 121.285 106.68 0)
-      (effects (font (size 1.27 1.27)) (justify left))
-    )
-    (property "Value" "4.7K" (at 125.73 113.03 90)
-      (effects (font (size 1.27 1.27)) (justify left))
-    )
-    (property "Footprint" "Resistor_SMD:R_0603_1608Metric_Pad0.98x0.95mm_HandSolder" (at 123.952 110.49 90)
-      (effects (font (size 1.27 1.27)) hide)
-    )
-    (property "Datasheet" "~" (at 125.73 110.49 0)
-      (effects (font (size 1.27 1.27)) hide)
-    )
-    (property "man" "yageo" (at 125.73 110.49 0)
-      (effects (font (size 1.27 1.27)) hide)
-    )
-    (property "man_no" "RC0603JR-0768RL" (at 125.73 110.49 0)
-      (effects (font (size 1.27 1.27)) hide)
-    )
-    (property "disti" "digikey" (at 125.73 110.49 0)
-      (effects (font (size 1.27 1.27)) hide)
-    )
-    (property "disti_no" "311-68GRTR-ND" (at 125.73 110.49 0)
-      (effects (font (size 1.27 1.27)) hide)
-    )
-    (pin "1")
-    (pin "2")
-    (instances
-      (project "ReflowController"
-        (path "/2394cc2a-b9b0-4c0b-be11-1fc6085b0d5c/c76c60d6-41ab-4683-93d6-43449ec74daf"
-          (reference "R606") (unit 1)
         )
       )
@@
         )
       )
-    )
-  )
-  (symbol (lib_id "Device:LED") (at 125.73 119.38 90) (unit 1)
-    (in_bom yes) (on_board yes) (dnp no)
-    (property "Reference" "D603" (at 121.92 116.84 90)
-      (effects (font (size 1.27 1.27)) (justify right))
-    )
-    (property "Value" "BLUE" (at 125.73 127 0)
-      (effects (font (size 1.27 1.27)) (justify right))
-    )
-    (property "Footprint" "LED_SMD:LED_0603_1608Metric_Pad1.05x0.95mm_HandSolder" (at 125.73 119.38 0)
-      (effects (font (size 1.27 1.27)) hide)
-    )
-    (property "Datasheet" "~" (at 125.73 119.38 0)
-      (effects (font (size 1.27 1.27)) hide)
-    )
-    (property "man" "lite-on" (at 125.73 119.38 90)
-      (effects (font (size 1.27 1.27)) hide)
-    )
-    (property "man_no" "LTST-C193TBKT-5A" (at 125.73 119.38 90)
-      (effects (font (size 1.27 1.27)) hide)
-    )
-    (property "dsiti" "digikey" (at 125.73 119.38 90)
-      (effects (font (size 1.27 1.27)) hide)
-    )
-    (property "disti_no" "160-1827-2-ND" (at 125.73 119.38 90)
-      (effects (font (size 1.27 1.27)) hide)
-    )
-    (pin "1")
-    (pin "2")
-    (instances
-      (project "ReflowController"
-        (path "/2394cc2a-b9b0-4c0b-be11-1fc6085b0d5c/c76c60d6-41ab-4683-93d6-43449ec74daf"
-          (reference "D603") (unit 1)
-        )
-      )

Commit message: changed port table + updated schema
Connections:
- net OI_AUX_1 renamed IO_AUX_1
- net OI_AUX_2 renamed IO_AUX_2
- net OI_AUX_3 renamed IO_AUX_3
- net OI_AUX_4 renamed IO_AUX_4
Changed lines of the file:
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@@
     (effects (font (size 1.27 1.27)) (justify left))
   )
-  (hierarchical_label "OI_AUX_3" (shape bidirectional) (at 67.945 140.335 0) (fields_autoplaced)
+  (hierarchical_label "IO_AUX_3" (shape bidirectional) (at 67.945 140.335 0) (fields_autoplaced)
     (effects (font (size 1.27 1.27)) (justify left))
   )
@@
     (effects (font (size 1.27 1.27)) (justify right))
   )
-  (hierarchical_label "OI_AUX_4" (shape bidirectional) (at 37.465 145.415 180) (fields_autoplaced)
+  (hierarchical_label "IO_AUX_4" (shape bidirectional) (at 37.465 145.415 180) (fields_autoplaced)
     (effects (font (size 1.27 1.27)) (justify right))
   )
@@
     (effects (font (size 1.27 1.27)) (justify right))
   )
-  (hierarchical_label "OI_AUX_2" (shape bidirectional) (at 67.945 142.875 0) (fields_autoplaced)
+  (hierarchical_label "IO_AUX_2" (shape bidirectional) (at 67.945 142.875 0) (fields_autoplaced)
     (effects (font (size 1.27 1.27)) (justify left))
   )
@@
     (effects (font (size 1.27 1.27)) (justify right))
   )
-  (hierarchical_label "OI_AUX_1" (shape bidirectional) (at 67.945 145.415 0) (fields_autoplaced)
+  (hierarchical_label "IO_AUX_1" (shape bidirectional) (at 67.945 145.415 0) (fields_autoplaced)
     (effects (font (size 1.27 1.27)) (justify left))
   )

Commit message: work on layout
Parts:
- added R1, R2: 4.7K, Resistor_SMD:R_0603_1608Metric_Pad0.98x0.95mm_HandSolder, symbol Device:R
Connections:
- net +3.3VD: now also R1.1, R2.1
- net SCL: now also R2.2
- net SDA: now also R1.2
Changed lines of the file:
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@@
   (junction (at 61.595 45.085) (diameter 0) (color 0 0 0 0)
   )
+  (junction (at 74.295 126.365) (diameter 0) (color 0 0 0 0)
+  )
   (junction (at 40.64 104.775) (diameter 0) (color 0 0 0 0)
   )
@@
   (junction (at 251.46 42.545) (diameter 0) (color 0 0 0 0)
   )
+  (junction (at 67.31 123.825) (diameter 0) (color 0 0 0 0)
+  )
   (junction (at 149.86 42.545) (diameter 0) (color 0 0 0 0)
   )
@@
   (junction (at 94.615 52.705) (diameter 0) (color 0 0 0 0)
   )
+  (wire (pts (xy 74.295 108.585) (xy 74.295 111.125))
+    (stroke (width 0) (type default))
+  )
   (wire (pts (xy 231.14 42.545) (xy 231.14 43.815))
     (stroke (width 0) (type default))
@@
     (stroke (width 0) (type default))
   )
+  (wire (pts (xy 67.31 118.745) (xy 67.31 123.825))
+    (stroke (width 0) (type default))
+  )
   (wire (pts (xy 37.465 135.255) (xy 40.005 135.255))
     (stroke (width 0) (type default))
@@
     (stroke (width 0) (type default))
   )
+  (wire (pts (xy 67.31 123.825) (xy 76.2 123.825))
+    (stroke (width 0) (type default))
+  )
   (wire (pts (xy 149.86 52.705) (xy 149.86 51.435))
     (stroke (width 0) (type default))
@@
     (stroke (width 0) (type default))
   )
-  (wire (pts (xy 65.405 123.825) (xy 68.58 123.825))
+  (wire (pts (xy 65.405 123.825) (xy 67.31 123.825))
     (stroke (width 0) (type default))
   )
@@
     (stroke (width 0) (type default))
   )
+  (wire (pts (xy 74.295 118.745) (xy 74.295 126.365))
+    (stroke (width 0) (type default))
+  )
   (wire (pts (xy 149.86 32.385) (xy 170.18 32.385))
     (stroke (width 0) (type default))
@@
     (stroke (width 0) (type default))
   )
-  (wire (pts (xy 65.405 126.365) (xy 68.58 126.365))
+  (wire (pts (xy 65.405 126.365) (xy 74.295 126.365))
     (stroke (width 0) (type default))
   )
@@
     (stroke (width 0) (type default))
   )
+  (wire (pts (xy 74.295 126.365) (xy 76.2 126.365))
+    (stroke (width 0) (type default))
+  )
   (wire (pts (xy 149.86 42.545) (xy 153.67 42.545))
     (stroke (width 0) (type default))
@@
   )
   (wire (pts (xy 234.95 42.545) (xy 234.95 56.515))
+    (stroke (width 0) (type default))
+  )
+  (wire (pts (xy 67.31 108.585) (xy 67.31 111.125))
     (stroke (width 0) (type default))
   )
@@
     (effects (font (size 1.27 1.27)) (justify right))
   )
+  (hierarchical_label "+3.3VD" (shape input) (at 74.295 108.585 90) (fields_autoplaced)
+    (effects (font (size 1.27 1.27)) (justify left))
+  )
   (hierarchical_label "DGND" (shape passive) (at 37.465 161.925 180) (fields_autoplaced)
     (effects (font (size 1.27 1.27)) (justify right))
@@
     (effects (font (size 1.27 1.27)) (justify right))
   )
-  (hierarchical_label "SDA" (shape bidirectional) (at 68.58 123.825 0) (fields_autoplaced)
+  (hierarchical_label "SDA" (shape bidirectional) (at 76.2 123.825 0) (fields_autoplaced)
     (effects (font (size 1.27 1.27)) (justify left))
   )
@@
     (effects (font (size 1.27 1.27)) (justify right))
   )
-  (hierarchical_label "SCL" (shape bidirectional) (at 68.58 126.365 0) (fields_autoplaced)
+  (hierarchical_label "SCL" (shape bidirectional) (at 76.2 126.365 0) (fields_autoplaced)
     (effects (font (size 1.27 1.27)) (justify left))
   )
@@
     (effects (font (size 1.27 1.27)) (justify right))
   )
+  (hierarchical_label "+3.3VD" (shape input) (at 67.31 108.585 90) (fields_autoplaced)
+    (effects (font (size 1.27 1.27)) (justify left))
+  )
   (symbol (lib_id "Device:C") (at 40.64 108.585 0) (unit 1)
     (in_bom yes) (on_board yes) (dnp no)
@@
   (symbol (lib_id "Device:R") (at 119.38 110.49 0) (unit 1)
     (in_bom yes) (on_board yes) (dnp no)
-    (property "Reference" "R605" (at 114.935 106.68 0)
+    (property "Reference" "R605" (at 121.285 108.585 0)
       (effects (font (size 1.27 1.27)) (justify left))
     )
@@
   (symbol (lib_id "Device:R") (at 113.03 110.49 0) (unit 1)
     (in_bom yes) (on_board yes) (dnp no)
-    (property "Reference" "R604" (at 107.95 107.315 0)
+    (property "Reference" "R604" (at 106.68 108.585 0)
       (effects (font (size 1.27 1.27)) (justify left))
     )
@@
     )
   )
+  (symbol (lib_id "Device:R") (at 74.295 114.935 0) (unit 1)
+    (in_bom yes) (on_board yes) (dnp yes)
+    (property "Reference" "R2" (at 69.215 111.76 0)
+      (effects (font (size 1.27 1.27)) (justify left))
+    )
+    (property "Value" "4.7K" (at 74.295 117.475 90)
+      (effects (font (size 1.27 1.27)) (justify left))
+    )
+    (property "Footprint" "Resistor_SMD:R_0603_1608Metric_Pad0.98x0.95mm_HandSolder" (at 72.517 114.935 90)
+      (effects (font (size 1.27 1.27)) hide)
+    )
+    (property "Datasheet" "~" (at 74.295 114.935 0)
+      (effects (font (size 1.27 1.27)) hide)
+    )
+    (property "man" "yageo" (at 74.295 114.935 0)
+      (effects (font (size 1.27 1.27)) hide)
+    )
+    (property "man_no" "RC0603JR-0768RL" (at 74.295 114.935 0)
+      (effects (font (size 1.27 1.27)) hide)
+    )
+    (property "disti" "digikey" (at 74.295 114.935 0)
+      (effects (font (size 1.27 1.27)) hide)
+    )
+    (property "disti_no" "311-68GRTR-ND" (at 74.295 114.935 0)
+      (effects (font (size 1.27 1.27)) hide)
+    )
+    (pin "1")
+    (pin "2")
+    (instances
+      (project "ReflowController"
+        (path "/2394cc2a-b9b0-4c0b-be11-1fc6085b0d5c/c76c60d6-41ab-4683-93d6-43449ec74daf"
+          (reference "R2") (unit 1)
+        )
+      )
+    )
+  )
   (symbol (lib_id "Device:C") (at 149.86 47.625 0) (unit 1)
     (in_bom yes) (on_board yes) (dnp no)
@@
         )
       )
+    )
+  )
+  (symbol (lib_id "Device:R") (at 67.31 114.935 0) (unit 1)
+    (in_bom yes) (on_board yes) (dnp yes)
+    (property "Reference" "R1" (at 62.23 111.76 0)
+      (effects (font (size 1.27 1.27)) (justify left))
+    )
+    (property "Value" "4.7K" (at 67.31 117.475 90)
+      (effects (font (size 1.27 1.27)) (justify left))
+    )
+    (property "Footprint" "Resistor_SMD:R_0603_1608Metric_Pad0.98x0.95mm_HandSolder" (at 65.532 114.935 90)
+      (effects (font (size 1.27 1.27)) hide)
+    )
+    (property "Datasheet" "~" (at 67.31 114.935 0)
+      (effects (font (size 1.27 1.27)) hide)
+    )
+    (property "man" "yageo" (at 67.31 114.935 0)
+      (effects (font (size 1.27 1.27)) hide)
+    )
+    (property "man_no" "RC0603JR-0768RL" (at 67.31 114.935 0)
+      (effects (font (size 1.27 1.27)) hide)
+    )
+    (property "disti" "digikey" (at 67.31 114.935 0)
+      (effects (font (size 1.27 1.27)) hide)
+    )
+    (property "disti_no" "311-68GRTR-ND" (at 67.31 114.935 0)
+      (effects (font (size 1.27 1.27)) hide)
+    )
+    (pin "1")
+    (pin "2")
+    (instances
+      (project "ReflowController"
+        (path "/2394cc2a-b9b0-4c0b-be11-1fc6085b0d5c/c76c60d6-41ab-4683-93d6-43449ec74daf"
+          (reference "R1") (unit 1)
+        )
+      )

Commit message: work on completion for first proto
Parts:
- removed R1, R2: 4.7K, Resistor_SMD:R_0603_1608Metric_Pad0.98x0.95mm_HandSolder, symbol Device:R
- added R2 (x2): 4k7, Resistor_SMD:R_1206_3216Metric, symbol Device:R
Connections:
- net +3.3VD: now also R2.1, R2.1
- net SCL: now also R2.2
- net SDA: now also R2.2
Changed lines of the file:
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@@
+    )
+  )
+  (symbol (lib_id "Device:R") (at 74.295 114.935 0) (unit 1)
+    (in_bom yes) (on_board yes) (dnp yes) (fields_autoplaced)
+    (property "Reference" "R2" (at 76.2 114.3 0)
+      (effects (font (size 1.27 1.27)) (justify left))
+    )
+    (property "Value" "4k7" (at 76.2 116.84 0)
+      (effects (font (size 1.27 1.27)) (justify left))
+    )
+    (property "Footprint" "Resistor_SMD:R_1206_3216Metric" (at 72.517 114.935 90)
+      (effects (font (size 1.27 1.27)) hide)
+    )
+    (property "Datasheet" "~" (at 74.295 114.935 0)
+      (effects (font (size 1.27 1.27)) hide)
+    )
+    (pin "1")
+    (pin "2")
+    (instances
+      (project "ReflowController"
+        (path "/2394cc2a-b9b0-4c0b-be11-1fc6085b0d5c/cedd135a-27b6-4ce6-9f5e-bdcd93291ccf"
+          (reference "R2") (unit 1)
+        )
+        (path "/2394cc2a-b9b0-4c0b-be11-1fc6085b0d5c/7f3c5223-ce8d-4c24-a6f4-4e6402f9b436"
+          (reference "R23") (unit 1)
+        )
+        (path "/2394cc2a-b9b0-4c0b-be11-1fc6085b0d5c/c76c60d6-41ab-4683-93d6-43449ec74daf"
+          (reference "R2") (unit 1)
+        )
+      )
     )
   )
@@
         (path "/e04c3b05-1837-4a0b-becb-f8e46c954cc1"
           (reference "BZ1") (unit 1)
+        )
+      )
+    )
+  )
+  (symbol (lib_id "Device:R") (at 67.31 114.935 0) (unit 1)
+    (in_bom yes) (on_board yes) (dnp yes)
+    (property "Reference" "R2" (at 62.23 114.3 0)
+      (effects (font (size 1.27 1.27)) (justify left))
+    )
+    (property "Value" "4k7" (at 62.23 116.84 0)
+      (effects (font (size 1.27 1.27)) (justify left))
+    )
+    (property "Footprint" "Resistor_SMD:R_1206_3216Metric" (at 65.532 114.935 90)
+      (effects (font (size 1.27 1.27)) hide)
+    )
+    (property "Datasheet" "~" (at 67.31 114.935 0)
+      (effects (font (size 1.27 1.27)) hide)
+    )
+    (pin "1")
+    (pin "2")
+    (instances
+      (project "ReflowController"
+        (path "/2394cc2a-b9b0-4c0b-be11-1fc6085b0d5c/cedd135a-27b6-4ce6-9f5e-bdcd93291ccf"
+          (reference "R2") (unit 1)
+        )
+        (path "/2394cc2a-b9b0-4c0b-be11-1fc6085b0d5c/7f3c5223-ce8d-4c24-a6f4-4e6402f9b436"
+          (reference "R23") (unit 1)
+        )
+        (path "/2394cc2a-b9b0-4c0b-be11-1fc6085b0d5c/c76c60d6-41ab-4683-93d6-43449ec74daf"
+          (reference "R1") (unit 1)
         )
       )
@@
     )
   )
-  (symbol (lib_id "Device:R") (at 74.295 114.935 0) (unit 1)
-    (in_bom yes) (on_board yes) (dnp yes)
-    (property "Reference" "R2" (at 69.215 111.76 0)
-      (effects (font (size 1.27 1.27)) (justify left))
-    )
-    (property "Value" "4.7K" (at 74.295 117.475 90)
-      (effects (font (size 1.27 1.27)) (justify left))
-    )
-    (property "Footprint" "Resistor_SMD:R_0603_1608Metric_Pad0.98x0.95mm_HandSolder" (at 72.517 114.935 90)
-      (effects (font (size 1.27 1.27)) hide)
-    )
-    (property "Datasheet" "~" (at 74.295 114.935 0)
-      (effects (font (size 1.27 1.27)) hide)
-    )
-    (property "man" "yageo" (at 74.295 114.935 0)
-      (effects (font (size 1.27 1.27)) hide)
-    )
-    (property "man_no" "RC0603JR-0768RL" (at 74.295 114.935 0)
-      (effects (font (size 1.27 1.27)) hide)
-    )
-    (property "disti" "digikey" (at 74.295 114.935 0)
-      (effects (font (size 1.27 1.27)) hide)
-    )
-    (property "disti_no" "311-68GRTR-ND" (at 74.295 114.935 0)
-      (effects (font (size 1.27 1.27)) hide)
-    )
-    (pin "1")
-    (pin "2")
-    (instances
-      (project "ReflowController"
-        (path "/2394cc2a-b9b0-4c0b-be11-1fc6085b0d5c/c76c60d6-41ab-4683-93d6-43449ec74daf"
-          (reference "R2") (unit 1)
-        )
-      )
-    )
-  )
   (symbol (lib_id "Device:C") (at 149.86 47.625 0) (unit 1)
     (in_bom yes) (on_board yes) (dnp no)
@@
         )
       )
-    )
-  )
-  (symbol (lib_id "Device:R") (at 67.31 114.935 0) (unit 1)
-    (in_bom yes) (on_board yes) (dnp yes)
-    (property "Reference" "R1" (at 62.23 111.76 0)
-      (effects (font (size 1.27 1.27)) (justify left))
-    )
-    (property "Value" "4.7K" (at 67.31 117.475 90)
-      (effects (font (size 1.27 1.27)) (justify left))
-    )
-    (property "Footprint" "Resistor_SMD:R_0603_1608Metric_Pad0.98x0.95mm_HandSolder" (at 65.532 114.935 90)
-      (effects (font (size 1.27 1.27)) hide)
-    )
-    (property "Datasheet" "~" (at 67.31 114.935 0)
-      (effects (font (size 1.27 1.27)) hide)
-    )
-    (property "man" "yageo" (at 67.31 114.935 0)
-      (effects (font (size 1.27 1.27)) hide)
-    )
-    (property "man_no" "RC0603JR-0768RL" (at 67.31 114.935 0)
-      (effects (font (size 1.27 1.27)) hide)
-    )
-    (property "disti" "digikey" (at 67.31 114.935 0)
-      (effects (font (size 1.27 1.27)) hide)
-    )
-    (property "disti_no" "311-68GRTR-ND" (at 67.31 114.935 0)
-      (effects (font (size 1.27 1.27)) hide)
-    )
-    (pin "1")
-    (pin "2")
-    (instances
-      (project "ReflowController"
-        (path "/2394cc2a-b9b0-4c0b-be11-1fc6085b0d5c/c76c60d6-41ab-4683-93d6-43449ec74daf"
-          (reference "R1") (unit 1)
-        )
-      )
