File: Hardware/ReflowController/ui.kicad_sch (KiCad schematic)
At the start: 44 parts, among them J601 LCD_HEADER, Q601 BC848, SW601 RotaryEncoder_Switch, SW602 SW_UP, SW603 SW_DOWN, SW604 SW_LEFT, SW605 SW_RIGHT, SW606 SW_SELECT, SW607 SW_RET, SW608 SW_RESET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

Commit message: work on BOM cleanup
Parts:
- removed R604, R605: 4.7K, Resistor_SMD:R_0603_1608Metric_Pad0.98x0.95mm_HandSolder, symbol Device:R
- added R2 (x2): 4k7, Resistor_SMD:R_1206_3216Metric, symbol Device:R
- BZ601: Dist Digikey -> (none); Dist no 445-2525-3-ND -> (none); Man TDK -> (none); Man no PS1240P02BT -> (none); disti (none) -> digikey; disti_no (none) -> 445-2525-3-ND; man (none) -> TDK; man_no (none) -> PS1240P02BT
- D601, D602: disti (none) -> digikey; dsiti digikey -> (none)
- Q601: Dist Digikey -> (none); Dist no 1727-4241-1-ND -> (none); Man Nexperia -> (none); Man no BC848B,215 -> (none); disti (none) -> digikey; disti_no (none) -> 1727-4241-1-ND; man (none) -> Nexperia; man_no (none) -> BC848B,215
Connections:
- net LED_ALIVE: now also R2.1
- net LED_ERROR: now also R2.1
- net at D602.2 (A): now also R2.2
- net at D601.2 (A): now also R2.2
Changed lines of the file:
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@@
       (effects (font (size 1.27 1.27)) hide)
     )
-    (property "dsiti" "digikey" (at 119.38 119.38 90)
+    (property "dsiti" "" (at 119.38 119.38 90)
       (effects (font (size 1.27 1.27)) hide)
     )
     (property "disti_no" "160-1446-2-ND" (at 119.38 119.38 90)
+      (effects (font (size 1.27 1.27)) hide)
+    )
+    (property "disti" "digikey" (at 119.38 119.38 0)
       (effects (font (size 1.27 1.27)) hide)
     )
@@
     )
   )
-  (symbol (lib_id "Device:R") (at 119.38 110.49 0) (unit 1)
-    (in_bom yes) (on_board yes) (dnp no)
-    (property "Reference" "R605" (at 121.285 108.585 0)
-      (effects (font (size 1.27 1.27)) (justify left))
-    )
-    (property "Value" "4.7K" (at 119.38 113.03 90)
-      (effects (font (size 1.27 1.27)) (justify left))
-    )
-    (property "Footprint" "Resistor_SMD:R_0603_1608Metric_Pad0.98x0.95mm_HandSolder" (at 117.602 110.49 90)
-      (effects (font (size 1.27 1.27)) hide)
-    )
-    (property "Datasheet" "~" (at 119.38 110.49 0)
-      (effects (font (size 1.27 1.27)) hide)
-    )
-    (property "man" "yageo" (at 119.38 110.49 0)
-      (effects (font (size 1.27 1.27)) hide)
-    )
-    (property "man_no" "RC0603JR-0768RL" (at 119.38 110.49 0)
-      (effects (font (size 1.27 1.27)) hide)
-    )
-    (property "disti" "digikey" (at 119.38 110.49 0)
-      (effects (font (size 1.27 1.27)) hide)
-    )
-    (property "disti_no" "311-68GRTR-ND" (at 119.38 110.49 0)
-      (effects (font (size 1.27 1.27)) hide)
-    )
-    (pin "1")
-    (pin "2")
-    (instances
-      (project "ReflowController"
-        (path "/2394cc2a-b9b0-4c0b-be11-1fc6085b0d5c/c76c60d6-41ab-4683-93d6-43449ec74daf"
-          (reference "R605") (unit 1)
-        )
-      )
-    )
-  )
   (symbol (lib_id "Device:Buzzer") (at 200.025 109.22 0) (unit 1)
     (in_bom yes) (on_board yes) (dnp no)
@@
       (effects (font (size 1.27 1.27)) hide)
     )
-    (property "Man" "TDK" (at 200.025 109.22 0)
-      (effects (font (size 1.27 1.27)) hide)
-    )
-    (property "Man no" "PS1240P02BT" (at 200.025 109.22 0)
-      (effects (font (size 1.27 1.27)) hide)
-    )
-    (property "Dist" "Digikey" (at 200.025 109.22 0)
-      (effects (font (size 1.27 1.27)) hide)
-    )
-    (property "Dist no" "445-2525-3-ND" (at 200.025 109.22 0)
+    (property "Man" "" (at 200.025 109.22 0)
+      (effects (font (size 1.27 1.27)) hide)
+    )
+    (property "Man no" "" (at 200.025 109.22 0)
+      (effects (font (size 1.27 1.27)) hide)
+    )
+    (property "Dist" "" (at 200.025 109.22 0)
+      (effects (font (size 1.27 1.27)) hide)
+    )
+    (property "Dist no" "" (at 200.025 109.22 0)
+      (effects (font (size 1.27 1.27)) hide)
+    )
+    (property "disti" "digikey" (at 200.025 109.22 0)
+      (effects (font (size 1.27 1.27)) hide)
+    )
+    (property "disti_no" "445-2525-3-ND" (at 200.025 109.22 0)
+      (effects (font (size 1.27 1.27)) hide)
+    )
+    (property "man" "TDK" (at 200.025 109.22 0)
+      (effects (font (size 1.27 1.27)) hide)
+    )
+    (property "man_no" "PS1240P02BT" (at 200.025 109.22 0)
       (effects (font (size 1.27 1.27)) hide)
     )
@@
     )
   )
+  (symbol (lib_id "Device:R") (at 113.03 110.49 0) (unit 1)
+    (in_bom yes) (on_board yes) (dnp no)
+    (property "Reference" "R2" (at 106.68 109.22 0)
+      (effects (font (size 1.27 1.27)) (justify left))
+    )
+    (property "Value" "4k7" (at 106.68 111.76 0)
+      (effects (font (size 1.27 1.27)) (justify left))
+    )
+    (property "Footprint" "Resistor_SMD:R_1206_3216Metric" (at 111.252 110.49 90)
+      (effects (font (size 1.27 1.27)) hide)
+    )
+    (property "Datasheet" "~" (at 113.03 110.49 0)
+      (effects (font (size 1.27 1.27)) hide)
+    )
+    (pin "1")
+    (pin "2")
+    (instances
+      (project "ReflowController"
+        (path "/2394cc2a-b9b0-4c0b-be11-1fc6085b0d5c/cedd135a-27b6-4ce6-9f5e-bdcd93291ccf"
+          (reference "R2") (unit 1)
+        )
+        (path "/2394cc2a-b9b0-4c0b-be11-1fc6085b0d5c/7f3c5223-ce8d-4c24-a6f4-4e6402f9b436"
+          (reference "R23") (unit 1)
+        )
+        (path "/2394cc2a-b9b0-4c0b-be11-1fc6085b0d5c/c76c60d6-41ab-4683-93d6-43449ec74daf"
+          (reference "R604") (unit 1)
+        )
+      )
+    )
+  )
   (symbol (lib_id "Device:R") (at 67.31 114.935 0) (unit 1)
     (in_bom yes) (on_board yes) (dnp yes)
@@
       (effects (font (size 1.27 1.27)) hide)
     )
-    (property "dsiti" "digikey" (at 113.03 119.38 90)
+    (property "dsiti" "" (at 113.03 119.38 90)
       (effects (font (size 1.27 1.27)) hide)
     )
     (property "disti_no" "160-1447-2-ND" (at 113.03 119.38 90)
+      (effects (font (size 1.27 1.27)) hide)
+    )
+    (property "disti" "digikey" (at 113.03 119.38 0)
       (effects (font (size 1.27 1.27)) hide)
     )
@@
         (path "/2394cc2a-b9b0-4c0b-be11-1fc6085b0d5c/c76c60d6-41ab-4683-93d6-43449ec74daf"
           (reference "C608") (unit 1)
-        )
-      )
-    )
-  )
-  (symbol (lib_id "Device:R") (at 113.03 110.49 0) (unit 1)
-    (in_bom yes) (on_board yes) (dnp no)
-    (property "Reference" "R604" (at 106.68 108.585 0)
-      (effects (font (size 1.27 1.27)) (justify left))
-    )
-    (property "Value" "4.7K" (at 113.03 113.03 90)
-      (effects (font (size 1.27 1.27)) (justify left))
-    )
-    (property "Footprint" "Resistor_SMD:R_0603_1608Metric_Pad0.98x0.95mm_HandSolder" (at 111.252 110.49 90)
-      (effects (font (size 1.27 1.27)) hide)
-    )
-    (property "Datasheet" "~" (at 113.03 110.49 0)
-      (effects (font (size 1.27 1.27)) hide)
-    )
-    (property "man" "yageo" (at 113.03 110.49 0)
-      (effects (font (size 1.27 1.27)) hide)
-    )
-    (property "man_no" "RC0603JR-0768RL" (at 113.03 110.49 0)
-      (effects (font (size 1.27 1.27)) hide)
-    )
-    (property "disti" "digikey" (at 113.03 110.49 0)
-      (effects (font (size 1.27 1.27)) hide)
-    )
-    (property "disti_no" "311-68GRTR-ND" (at 113.03 110.49 0)
-      (effects (font (size 1.27 1.27)) hide)
-    )
-    (pin "1")
-    (pin "2")
-    (instances
-      (project "ReflowController"
-        (path "/2394cc2a-b9b0-4c0b-be11-1fc6085b0d5c/c76c60d6-41ab-4683-93d6-43449ec74daf"
-          (reference "R604") (unit 1)
         )
       )
@@
       (effects (font (size 1.27 1.27)) (justify left) hide)
     )
-    (property "Man" "Nexperia" (at 186.055 119.38 0)
-      (effects (font (size 1.27 1.27)) hide)
-    )
-    (property "Man no" "BC848B,215" (at 186.055 119.38 0)
-      (effects (font (size 1.27 1.27)) hide)
-    )
-    (property "Dist" "Digikey" (at 186.055 119.38 0)
-      (effects (font (size 1.27 1.27)) hide)
-    )
-    (property "Dist no" "1727-4241-1-ND" (at 186.055 119.38 0)
+    (property "Man" "" (at 186.055 119.38 0)
+      (effects (font (size 1.27 1.27)) hide)
+    )
+    (property "Man no" "" (at 186.055 119.38 0)
+      (effects (font (size 1.27 1.27)) hide)
+    )
+    (property "Dist" "" (at 186.055 119.38 0)
+      (effects (font (size 1.27 1.27)) hide)
+    )
+    (property "Dist no" "" (at 186.055 119.38 0)
+      (effects (font (size 1.27 1.27)) hide)
+    )
+    (property "disti" "digikey" (at 186.055 119.38 0)
+      (effects (font (size 1.27 1.27)) hide)
+    )
+    (property "disti_no" "1727-4241-1-ND" (at 186.055 119.38 0)
+      (effects (font (size 1.27 1.27)) hide)
+    )
+    (property "man" "Nexperia" (at 186.055 119.38 0)
+      (effects (font (size 1.27 1.27)) hide)
+    )
+    (property "man_no" "BC848B,215" (at 186.055 119.38 0)
       (effects (font (size 1.27 1.27)) hide)
     )
@@
         )
       )
+    )
+  )
+  (symbol (lib_id "Device:R") (at 119.38 110.49 0) (unit 1)
+    (in_bom yes) (on_board yes) (dnp no)
+    (property "Reference" "R2" (at 120.65 109.22 0)
+      (effects (font (size 1.27 1.27)) (justify left))
+    )
+    (property "Value" "4k7" (at 120.65 111.76 0)
+      (effects (font (size 1.27 1.27)) (justify left))
+    )
+    (property "Footprint" "Resistor_SMD:R_1206_3216Metric" (at 117.602 110.49 90)
+      (effects (font (size 1.27 1.27)) hide)
+    )
+    (property "Datasheet" "~" (at 119.38 110.49 0)
+      (effects (font (size 1.27 1.27)) hide)
+    )
+    (pin "1")
+    (pin "2")
+    (instances
+      (project "ReflowController"
+        (path "/2394cc2a-b9b0-4c0b-be11-1fc6085b0d5c/cedd135a-27b6-4ce6-9f5e-bdcd93291ccf"
+          (reference "R2") (unit 1)
+        )
+        (path "/2394cc2a-b9b0-4c0b-be11-1fc6085b0d5c/7f3c5223-ce8d-4c24-a6f4-4e6402f9b436"
+          (reference "R23") (unit 1)
+        )
+        (path "/2394cc2a-b9b0-4c0b-be11-1fc6085b0d5c/c76c60d6-41ab-4683-93d6-43449ec74daf"
+          (reference "R605") (unit 1)
+        )
+      )
